File: demo/demo.kicad_pcb (KiCad board)
At the start: 2 copper layers, 1206 parts

Commit message: Modify pads
Routing:
- net Net-(INV14-Pad1): track 387.7 -> 394.8 mm
- net Net-(INV10-Pad1): track 487.2 -> 488.0 mm
Changed lines of the file:
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@@
   (arc (start -63.743787 -87.303126) (mid -62.070694 -85.663659) (end -60.362401 -84.060905) (width 2) (layer "F.Cu") (net 4))
   (arc (start -12.513474 -35.72974) (mid -11.069965 -33.886093) (end -9.56602 -32.091405) (width 2) (layer "F.Cu") (net 4))
+  (segment (start 490.1 -187) (end 421.2 -149.6) (width 2) (layer "F.Cu") (net 5))
+  (segment (start 347.7 -109.1) (end 287.6 -87.937991) (width 2) (layer "F.Cu") (net 5))
+  (segment (start 68.724488 -22.080001) (end 46.398108 -14.89985) (width 2) (layer "F.Cu") (net 5))
+  (segment (start 288.9 -88.4) (end 287.6 -87.937991) (width 2) (layer "F.Cu") (net 5))
+  (segment (start 177.13584 -49.093905) (end 101.437619 -31.191031) (width 2) (layer "F.Cu") (net 5))
+  (segment (start 421.2 -149.6) (end 347.7 -109.1) (width 2) (layer "F.Cu") (net 5))
+  (segment (start 287.6 -87.937991) (end 181.664627 -50.289464) (width 2) (layer "F.Cu") (net 5))
   (segment (start 42.231318 -12.900945) (end 39.2 -10.9) (width 2) (layer "F.Cu") (net 5))
   (segment (start 96.900579 -30.023215) (end 73.211918 -23.425883) (width 2) (layer "F.Cu") (net 5))
-  (segment (start 301.85716 -86.142705) (end 490.1 -187) (width 2) (layer "F.Cu") (net 5))
-  (segment (start 46.398108 -14.89985) (end 68.724488 -22.080001) (width 2) (layer "F.Cu") (net 5))
-  (segment (start 297.072072 -83.971905) (end 181.664627 -50.289464) (width 2) (layer "F.Cu") (net 5))
-  (segment (start 101.437619 -31.191031) (end 177.13584 -49.093905) (width 2) (layer "F.Cu") (net 5))
+  (arc (start 46.398108 -14.89985) (mid 44.246574 -14.042435) (end 42.231318 -12.900945) (width 2) (layer "F.Cu") (net 5))
+  (arc (start 101.437619 -31.191031) (mid 99.16335 -30.629459) (end 96.900579 -30.023215) (width 2) (layer "F.Cu") (net 5))
   (arc (start 73.211918 -23.425883) (mid 70.961552 -22.775118) (end 68.724488 -22.080001) (width 2) (layer "F.Cu") (net 5))
   (arc (start 181.664627 -50.289464) (mid 179.407965 -49.662397) (end 177.13584 -49.093905) (width 2) (layer "F.Cu") (net 5))
-  (arc (start 101.437619 -31.191031) (mid 99.16335 -30.629459) (end 96.900579 -30.023215) (width 2) (layer "F.Cu") (net 5))
-  (arc (start 46.398108 -14.89985) (mid 44.246574 -14.042435) (end 42.231318 -12.900945) (width 2) (layer "F.Cu") (net 5))
-  (arc (start 301.85716 -86.142705) (mid 300.691027 -85.528451) (end 299.51635 -84.9307) (width 2) (layer "F.Cu") (net 5))
-  (arc (start 299.51635 -84.9307) (mid 298.315761 -84.396362) (end 297.072072 -83.971905) (width 2) (layer "F.Cu") (net 5))
   (segment (start 53.526122 0.215282) (end 39.1 -7.3) (width 2) (layer "F.Cu") (net 6))
   (segment (start 414.772177 152.801716) (end 235.284481 79.935547) (width 2) (layer "F.Cu") (net 6))
@@
   (arc (start 301.715908 -82.177462) (mid 299.489917 -81.44678) (end 297.274561 -80.684463) (width 2) (layer "F.Cu") (net 1182))
   (arc (start 414.289316 -118.179315) (mid 412.044572 -117.508286) (end 409.808772 -116.808032) (width 2) (layer "F.Cu") (net 1182))
-  (segment (start -156.943505 -100.195025) (end -264.094605 -157.513557) (width 2) (layer "F.Cu") (net 1183))
-  (segment (start -268.348865 -159.442747) (end -341.5 -187) (width 2) (layer "F.Cu") (net 1183))
+  (segment (start -29.089346 -31.254192) (end -24.8 -29.1) (width 2) (layer "F.Cu") (net 1183))
+  (segment (start -30.3 -33.4) (end -29.089346 -31.254192) (width 2) (layer "F.Cu") (net 1183))
+  (segment (start -24.8 -29.1) (end -27.823626 -30.57161) (width 2) (layer "F.Cu") (net 1183))
+  (segment (start -26.235409 -29.704078) (end -21.654932 -27.17008) (width 2) (layer "F.Cu") (net 1183))
+  (segment (start -264.094605 -157.513557) (end -156.943505 -100.195025) (width 2) (layer "F.Cu") (net 1183))
+  (segment (start -152.81504 -97.9776) (end -30.3 -33.4) (width 2) (layer "F.Cu") (net 1183))
+  (segment (start -341.5 -187) (end -268.348865 -159.442747) (width 2) (layer "F.Cu") (net 1183))
   (segment (start -17.656691 -24.737154) (end 3.1 -10.9) (width 2) (layer "F.Cu") (net 1183))
-  (segment (start -152.81504 -97.9776) (end -29.089346 -31.254192) (width 2) (layer "F.Cu") (net 1183))
-  (segment (start -21.654932 -27.17008) (end -24.976706 -29.007742) (width 2) (layer "F.Cu") (net 1183))
   (arc (start -156.943505 -100.195025) (mid -154.878336 -99.088056) (end -152.81504 -97.9776) (width 2) (layer "F.Cu") (net 1183))
-  (arc (start -29.089346 -31.254192) (mid -27.030013 -30.136483) (end -24.976706 -29.007742) (width 2) (layer "F.Cu") (net 1183))
   (arc (start -268.348865 -159.442747) (mid -266.190151 -158.547801) (end -264.094605 -157.513557) (width 2) (layer "F.Cu") (net 1183))
+  (arc (start -27.823626 -30.57161) (mid -27.028354 -30.139974) (end -26.235409 -29.704078) (width 2) (layer "F.Cu") (net 1183))
   (arc (start -21.654932 -27.17008) (mid -19.630666 -25.99494) (end -17.656691 -24.737154) (width 2) (layer "F.Cu") (net 1183))
   (segment (start -54.869927 -26.347717) (end -8.8 -10.9) (width 2) (layer "F.Cu") (net 1184))
